File: board/chrimbus2022.kicad_pcb (KiCad board)
At the start: 2 copper layers, 57.9 x 57.9 mm, 4 parts

Commit message: board finalized
Parts:
- added BT1: Battery_Cell, Battery:BatteryHolder_MPD_BC2003_1x2032, B.Cu at (139.1, 125.1)
- added D1: LED, toolbox-led:Kingbright_AA3528, B.Cu at (128.2, 102.2)
- added D2: LED, toolbox-led:Kingbright_AA3528, B.Cu at (147.3, 104.1)
- added H1: MountingHole_3.2M3, MountingHole:MountingHole_3.2mm_M3, B.Cu at (162.6, 116.8)
- added R1: R, Resistor_SMD:R_1206_3216Metric_Pad1.30x1.75mm_HandSolder, B.Cu at (125.1, 113.0)
- added R2: R, Resistor_SMD:R_1206_3216Metric_Pad1.30x1.75mm_HandSolder, B.Cu at (150.5, 113.0)
- added SW1: SW_SPDT, toolbox-switch:C&K_JS102011SCQN, B.Cu at (139.1, 92.1)
Routing:
- net Net-(SW1-Pad3): track 0.00 -> 85.3 mm
- net +3V3: track 0.00 -> 74.2 mm
- net GND: track 0.00 -> 53.7 mm
- net Net-(D1-Pad2): track 0.00 -> 11.7 mm
- net Net-(D2-Pad2): track 0.00 -> 10.7 mm
Other:
- board text added: "LOVE, JAKE"
- board text added: "MERRY CHRISTMAS 2022"
- board text added: "OFF"
- board text added: "ON"
